File: capkey.sch (KiCad schematic (older format))
At the start: 19 parts, among them J1 TIP, J2 RING, J3 AudioJack4, Q1 Q_NMOS_DGS, Q2 Q_NMOS_DGS, SW1 SW_SPDT, U1 AT42QT1011-TSHR, U2 AT42QT1011-TSHR, U3 L78L05_SOT89

Commit message: switched paddle sides
Parts:
- removed JP1: SolderJumper_2_Open, Jumper:SolderJumper-2_P1.3mm_Open_RoundedPad1.0x1.5mm, symbol Jumper:SolderJumper_2_Open
- removed U3: L78L05_SOT89, Package_TO_SOT_SMD:SOT-89-3, symbol Regulator_Linear:L78L05_SOT89
- added LOGO1: dahu-logo, w6ipa-footprints:W6IPA-Logo-9mmx8mm, symbol w6ipa_graphic:dahu-logo
- Q1, Q2: value Q_NMOS_DGS -> IRFML8244TRPbF; symbol Device:Q_NMOS_DGS -> Device:Q_NMOS_GSD
Connections:
- net GND: now also Q1.2 (S), Q2.2 (S); no longer Q1.3 (S), Q2.3 (S)
- net ring: now also Q1.3 (D); no longer Q2.1 (D)
- net tip: now also Q2.3 (D); no longer Q1.1 (D)
- net at U2.1 (OUT): now also Q2.1 (G); no longer Q2.2 (G)
- net at C2.1, C3.1, U1.5 (VDD)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: now also SW1.1 (A)
- net at U1.1 (OUT): now also Q1.1 (G); no longer Q1.2 (G)
Changed lines of the file:
@@
 EESchema Schematic File Version 4
+LIBS:capkey-cache
 EELAYER 30 0
 EELAYER END
@@
 Comment4 ""
 $EndDescr
+Text GLabel 8150 2600 2    50   Input ~ 0
+tip
+Wire Wire Line
+	3250 2600 3500 2600
 Text GLabel 3250 2600 0    50   Input ~ 0
-tip
-Wire Wire Line
-	3250 2600 3500 2600
-Text GLabel 8150 2600 2    50   Input ~ 0
 ring
 Wire Wire Line
@@
 Wire Wire Line
 	5700 3800 6000 3800
-Connection ~ 5750 2800
-Wire Wire Line
-	5750 2800 6000 2800
 Wire Wire Line
 	5250 3100 5250 2800
 Connection ~ 5250 2800
-Wire Wire Line
-	5250 2800 5750 2800
 Wire Wire Line
 	5250 3400 5250 3800
@@
 Text GLabel 6300 2250 0    50   Input ~ 0
 tip
-$Comp
-L power:GND #PWR04
-U 1 1 5E3F5692
-P 5400 2300
-F 0 "#PWR04" H 5400 2050 50  0001 C CNN
-F 1 "GND" H 5405 2127 50  0000 C CNN
-F 2 "" H 5400 2300 50  0001 C CNN
-F 3 "" H 5400 2300 50  0001 C CNN
-	1    5400 2300
-	1    0    0    -1
-$EndComp
-Wire Wire Line
-	5400 2150 5400 2300
-Wire Wire Line
-	5000 1950 5000 1850
-Wire Wire Line
-	5000 1850 5100 1850
-Wire Wire Line
-	5750 1850 5700 1850
-Wire Wire Line
-	5750 1850 5750 2800
-Wire Wire Line
-	5000 1850 5000 1400
-Wire Wire Line
-	5000 1400 5250 1400
-Connection ~ 5000 1850
-Wire Wire Line
-	5550 1400 5750 1400
-Wire Wire Line
-	5750 1400 5750 1850
-Connection ~ 5750 1850
 Wire Wire Line
 	6450 1950 6850 1950
@@
 Wire Wire Line
 	6300 2250 6850 2250
-Wire Wire Line
-	5000 1850 4850 1850
-Connection ~ 3900 1950
 Wire Wire Line
 	3900 1950 4450 1950
@@
 $EndComp
 $Comp
-L Jumper:SolderJumper_2_Open JP1
-U 1 1 5E3FF1E1
-P 5400 1400
-F 0 "JP1" H 5400 1605 50  0000 C CNN
-F 1 "SolderJumper_2_Open" H 5400 1514 50  0000 C CNN
-F 2 "Jumper:SolderJumper-2_P1.3mm_Open_RoundedPad1.0x1.5mm" H 5400 1400 50  0001 C CNN
-F 3 "~" H 5400 1400 50  0001 C CNN
-	1    5400 1400
-	1    0    0    -1
-$EndComp
-$Comp
-L Regulator_Linear:L78L05_SOT89 U3
-U 1 1 5E3EEBE6
-P 5400 1850
-F 0 "U3" H 5400 2092 50  0000 C CNN
-F 1 "L78L05_SOT89" H 5400 2001 50  0000 C CNN
-F 2 "Package_TO_SOT_SMD:SOT-89-3" H 5400 2050 50  0001 C CIN
-F 3 "http://www.st.com/content/ccc/resource/technical/document/datasheet/15/55/e5/aa/23/5b/43/fd/CD00000446.pdf/files/CD00000446.pdf/jcr:content/translations/en.CD00000446.pdf" H 5400 1800 50  0001 C CNN
-	1    5400 1850
-	1    0    0    -1
-$EndComp
-$Comp
-L Device:Battery_Cell BT1
-U 1 1 5E3CC0F6
-P 3900 2150
-F 0 "BT1" H 4018 2246 50  0000 L CNN
-F 1 "Battery_Cell" H 4018 2155 50  0000 L CNN
-F 2 "Battery:BatteryHolder_Keystone_103_1x20mm" V 3900 2210 50  0001 C CNN
-F 3 "~" V 3900 2210 50  0001 C CNN
-	1    3900 2150
-	1    0    0    -1
-$EndComp
-$Comp
 L Device:C C3
 U 1 1 5E3C70D3
@@
 $EndComp
 $Comp
-L Device:Q_NMOS_DGS Q2
+L Device:Q_NMOS_GSD Q2
 U 1 1 5E336CA0
 P 7800 3150
 F 0 "Q2" H 8006 3196 50  0000 L CNN
-F 1 "Q_NMOS_DGS" H 8006 3105 50  0000 L CNN
+F 1 "IRFML8244TRPbF" H 8006 3105 50  0000 L CNN
 F 2 "Package_TO_SOT_SMD:SOT-23" H 8000 3250 50  0001 C CNN
 F 3 "~" H 7800 3150 50  0001 C CNN
@@
 $EndComp
 $Comp
-L Device:Q_NMOS_DGS Q1
+L Device:Q_NMOS_GSD Q1
 U 1 1 5E3343FB
 P 3600 3150
 F 0 "Q1" H 3806 3196 50  0000 L CNN
-F 1 "Q_NMOS_DGS" H 3806 3105 50  0000 L CNN
+F 1 "IRFML8244TRPbF" H 3806 3105 50  0000 L CNN
 F 2 "Package_TO_SOT_SMD:SOT-23" H 3800 3250 50  0001 C CNN
 F 3 "~" H 3600 3150 50  0001 C CNN
@@
 	0    1    1    0
 $EndComp
+Wire Wire Line
+	5250 2800 5650 2800
+Wire Wire Line
+	4850 1850 5650 1850
+Wire Wire Line
+	5650 1850 5650 2800
+Connection ~ 5650 2800
+Wire Wire Line
+	5650 2800 6000 2800
+$Comp
+L w6ipa_graphic:dahu-logo LOGO1
+U 1 1 5E3CD739
+P 7450 6800
+F 0 "LOGO1" H 7475 6846 50  0000 L CNN
+F 1 "dahu-logo" H 7475 6755 50  0000 L CNN
+F 2 "w6ipa-footprints:W6IPA-Logo-9mmx8mm" H 7450 6900 50  0001 C CNN
+F 3 "" H 7450 6900 50  0001 C CNN
+	1    7450 6800
+	1    0    0    -1
+$EndComp
+Connection ~ 3900 1950
+$Comp
+L Device:Battery_Cell BT1
+U 1 1 5E3CC0F6
+P 3900 2150
+F 0 "BT1" H 4018 2246 50  0000 L CNN
+F 1 "Battery_Cell" H 4018 2155 50  0000 L CNN
+F 2 "Battery:BatteryHolder_Keystone_103_1x20mm" V 3900 2210 50  0001 C CNN
+F 3 "~" V 3900 2210 50  0001 C CNN
+	1    3900 2150
+	1    0    0    -1
+$EndComp
 $EndSCHEMATC
